Commit message: Added casters in the urdf

File: fetch_description/robots/fetch.urdf (robot description, URDF)
Before this commit: robot fetch, 26 links, 25 joints
Links:
- added link bl_caster_link
- added link br_caster_link
- added link fl_caster_link
- added link fr_caster_link
Joints:
- added joint bl_caster_joint: type fixed, parent base_link, child bl_caster_link
- added joint br_caster_joint: type fixed, parent base_link, child br_caster_link
- added joint fl_caster_joint: type fixed, parent base_link, child fl_caster_link
- added joint fr_caster_joint: type fixed, parent base_link, child fr_caster_link

Commit message: Removed casters from urdf

File: fetch_description/robots/fetch.urdf (robot description, URDF)
Before this commit: robot fetch, 30 links, 29 joints
Links:
- removed link bl_caster_link
- removed link br_caster_link
- removed link fl_caster_link
- removed link fr_caster_link
Joints:
- removed joint bl_caster_joint
- removed joint br_caster_joint
- removed joint fl_caster_joint
- removed joint fr_caster_joint
